Commit message: Add MoveIt config files for Spot

File: src/spot_skills/urdf/spot_with_arm.urdf (robot description, URDF)
Before this commit: robot spot, 26 links, 25 joints
Links:
- link body: mass None -> 0.1
- link front_left_hip: mass None -> 0.1
- link front_left_lower_leg: mass None -> 0.1
- link front_left_upper_leg: mass None -> 0.1
- link front_right_hip: mass None -> 0.1
- link front_right_lower_leg: mass None -> 0.1
- link front_right_upper_leg: mass None -> 0.1
- link rear_left_hip: mass None -> 0.1
- link rear_left_lower_leg: mass None -> 0.1
- link rear_left_upper_leg: mass None -> 0.1
- link rear_right_hip: mass None -> 0.1
- link rear_right_lower_leg: mass None -> 0.1
- link rear_right_upper_leg: mass None -> 0.1

Commit message: Clean up Spot's leg joint limits and defaults

File: src/spot_skills/urdf/spot_with_arm.urdf (robot description, URDF)
Before this commit: robot spot, 26 links, 25 joints
Joints:
- joint front_left_knee: limit lower=-2.7929 upper=-0.254801 effort=1000 velocity=1000.00 -> lower=-2.79253 upper=-0.261799 effort=1000 velocity=1000.00
- joint front_right_knee: limit lower=-2.7929 upper=-0.247563 effort=1000 velocity=1000.00 -> lower=-2.79253 upper=-0.261799 effort=1000 velocity=1000.00
- joint rear_left_knee: limit lower=-2.7929 upper=-0.267153 effort=1000 velocity=1000.00 -> lower=-2.79253 upper=-0.261799 effort=1000 velocity=1000.00
- joint rear_right_knee: limit lower=-2.7929 upper=-0.257725 effort=1000 velocity=1000.00 -> lower=-2.79253 upper=-0.261799 effort=1000 velocity=1000.00

Commit message: Update URDF to version based on spot_ros2

File: src/spot_skills/urdf/spot_with_arm.urdf (robot description, URDF)
Before this commit: robot spot, 26 links, 25 joints
Links:
- removed link base_arm_link
- removed link finger
- removed link gripper
- removed link link1
- removed link link2
- removed link link3
- removed link link4
- removed link real_front_rail
- removed link real_rear_rail
- removed link wrist
- added link arm_link_el0, mass 0.725; collision mesh filename=package://spot_description/meshes/arm/collision/arm_link_el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; visual mesh filename=package://spot_description/meshes/arm/visual/arm_link_el0.o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
- added link arm_link_el1, mass 0.725; collision mesh filename=package://spot_description/meshes/arm/collision/arm_link_el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; collision mesh filename=package://spot_description/meshes/arm/collision/arm_link_el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
- added link arm_link_fngr, mass 0.2; collision mesh filename=package://spot_description/meshes/arm/collision/left_finger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; collision mesh filename=package://spot_description/meshes/arm/collision/left_hinge.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
- added link arm_link_hr0, mass 1e-06; collision mesh filename=package://spot_description/meshes/arm/collision/arm_link_hr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; visual mesh filename=package://spot_description/meshes/arm/visual/arm_link_hr0.o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
- added link arm_link_sh0, mass 2.3364000000000003; collision mesh filename=package://spot_description/meshes/arm/collision/arm_link_sh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; collision mesh filename=package://spot_description/meshes/arm/collision/arm_link_sh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
- added link arm_link_sh1, mass 0.2596; visual mesh filename=package://spot_description/meshes/arm/visual/arm_link_sh1.o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
- added link arm_link_wr0, mass 0.98; collision mesh filename=package://spot_description/meshes/arm/collision/arm_link_wr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; visual mesh filename=package://spot_description/meshes/arm/visual/arm_link_wr0.o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
- added link arm_link_wr1, mass 0.785; collision mesh filename=package://spot_description/meshes/arm/collision/arm_link_wr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; collision mesh filename=package://spot_description/meshes/arm/collision/front_jaw.o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
- link base_link: mass None -> 32.86
- link body: mass 0.1 -> None; geometry collision mesh filename=package://spot_description/meshes/base/collision/body_colli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; visual mesh filename=package://spot_description/meshes/base/visual/body.obj
- link front_left_hip: mass 0.1 -> 1.68; geometry visual mesh filename=package://spot_description/meshes/base/visual/front_left_hi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
- link front_left_lower_leg: mass 0.1 -> 0.35; geometry collision mesh filename=package://spot_description/meshes/base/collision/left_lower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; collision sphere radius=0.036
- link front_left_upper_leg: mass 0.1 -> 2.34; geometry collision mesh filename=package://spot_description/meshes/base/collision/left_upper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; visual mesh filename=package://spot_description/meshes/base/visual/front_left_up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
- link front_rail: mass None -> 1.0e-6
- link front_right_hip: mass 0.1 -> 1.68; geometry visual mesh filename=package://spot_description/meshes/base/visual/front_right_h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
- link front_right_lower_leg: mass 0.1 -> 0.35; geometry collision mesh filename=package://spot_description/meshes/base/collision/right_lowe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; collision sphere radius=0.036
- link front_right_upper_leg: mass 0.1 -> 2.34; geometry collision mesh filename=package://spot_description/meshes/base/collision/right_uppe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; visual mesh filename=package://spot_description/meshes/base/visual/front_right_u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
- link rear_left_hip: mass 0.1 -> 1.68; geometry visual mesh filename=package://spot_description/meshes/base/visual/rear_left_hip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
- link rear_left_lower_leg: mass 0.1 -> 0.35; geometry collision mesh filename=package://spot_description/meshes/base/collision/left_lower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; collision sphere radius=0.036
- link rear_left_upper_leg: mass 0.1 -> 2.34; geometry collision mesh filename=package://spot_description/meshes/base/collision/left_upper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; visual mesh filename=package://spot_description/meshes/base/visual/rear_left_upp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
- link rear_rail: mass None -> 1.0e-6
- link rear_right_hip: mass 0.1 -> 1.68; geometry visual mesh filename=package://spot_description/meshes/base/visual/rear_right_hi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
- link rear_right_lower_leg: mass 0.1 -> 0.35; geometry collision mesh filename=package://spot_description/meshes/base/collision/right_lowe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; collision sphere radius=0.036
- link rear_right_upper_leg: mass 0.1 -> 2.34; geometry collision mesh filename=package://spot_description/meshes/base/collision/right_uppe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; visual mesh filename=package://spot_description/meshes/base/visual/rear_right_up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
Joints:
- removed joint arm_gripper
- removed joint arm_joint1
- removed joint arm_joint2
- removed joint arm_joint3
- removed joint arm_joint4
- removed joint arm_joint5
- removed joint arm_joint6
- removed joint base_arm_joint
- removed joint real_front_rail_joint
- removed joint real_rear_rail_joint
- added joint arm_el0: type revolute, parent arm_link_hr0, child arm_link_el0, origin xyz=0.3385 0 0 rpy=0 0 0, axis 0 1 0, limit lower=0 upper=3.14159265358979311599 effort=90.9 velocity=10.0
- added joint arm_el1: type revolute, parent arm_link_el0, child arm_link_el1, origin xyz=0.40330 0.0 0.0750 rpy=0 0 0, axis 1 0 0, limit lower=-2.79252680319092716487 upper=2.79252680319092716487 effort=30.3 velocity=10.0
- added joint arm_f1x: type revolute, parent arm_link_wr1, child arm_link_fngr, origin xyz=0.11745 0 0.014820 rpy=0 0 0, axis 0.0 1.0 0.0, limit lower=-1.57 upper=0.0 effort=15.32 velocity=10.0
- added joint arm_hr0: type fixed, parent arm_link_sh1, child arm_link_hr0, origin xyz=0.0 0.0 0.0 rpy=0 0 0
- added joint arm_sh0: type revolute, parent body, child arm_link_sh0, origin xyz=0.292 0.0 0.188 rpy=0 0 0, axis 0 0 1, limit lower=-2.61799387799149441136 upper=3.14159265358979311599 effort=90.9 velocity=10.0
- added joint arm_sh1: type revolute, parent arm_link_sh0, child arm_link_sh1, origin xyz=0.0 0.0 0.0 rpy=0 0 0, axis 0 1 0, limit lower=-3.14159265358979311599 upper=0.52359877559829881565 effort=181.8 velocity=10.0
- added joint arm_wr0: type revolute, parent arm_link_el1, child arm_link_wr0, origin xyz=0.0 0.0 0.0 rpy=0 0 0, axis 0 1 0, limit lower=-1.83259571459404613236 upper=1.83259571459404613236 effort=30.3 velocity=10.0
- added joint arm_wr1: type revolute, parent arm_link_wr0, child arm_link_wr1, origin xyz=0.0 0.0 0.0 rpy=0 0 0, axis 1 0 0, limit lower=-2.87979326579064354163 upper=2.87979326579064354163 effort=30.3 velocity=10.0
- joint front_left_hip_x: limit lower=-0.78539816339744827899 upper=0.78539816339744827899 effort=1000 velocity=1000.00 -> lower=-0.78539816339744827899 upper=0.78539816339744827899 effort=45 velocity=17.647
- joint front_left_hip_y: limit lower=-0.89884456477707963539 upper=2.2951079663725435509 effort=1000 velocity=1000.00 -> lower=-0.89884456477707963539 upper=2.2951079663725435509 effort=45 velocity=17.647
- joint front_left_knee: limit lower=-2.79253 upper=-0.261799 effort=1000 velocity=1000.00 -> lower=-2.7929 upper=-0.254801 effort=115 velocity=12.0
- joint front_right_hip_x: limit lower=-0.78539816339744827899 upper=0.78539816339744827899 effort=1000 velocity=1000.00 -> lower=-0.78539816339744827899 upper=0.78539816339744827899 effort=45 velocity=17.647
- joint front_right_hip_y: limit lower=-0.89884456477707963539 upper=2.2951079663725435509 effort=1000 velocity=1000.00 -> lower=-0.89884456477707963539 upper=2.2951079663725435509 effort=45 velocity=17.647
- joint front_right_knee: limit lower=-2.79253 upper=-0.261799 effort=1000 velocity=1000.00 -> lower=-2.7929 upper=-0.247563 effort=115 velocity=12.0
- joint rear_left_hip_x: limit lower=-0.78539816339744827899 upper=0.78539816339744827899 effort=1000 velocity=1000.00 -> lower=-0.78539816339744827899 upper=0.78539816339744827899 effort=45 velocity=17.647
- joint rear_left_hip_y: limit lower=-0.89884456477707963539 upper=2.2951079663725435509 effort=1000 velocity=1000.00 -> lower=-0.89884456477707963539 upper=2.2951079663725435509 effort=45 velocity=17.647
- joint rear_left_knee: limit lower=-2.79253 upper=-0.261799 effort=1000 velocity=1000.00 -> lower=-2.7929 upper=-0.267153 effort=115 velocity=12.0
- joint rear_right_hip_x: limit lower=-0.78539816339744827899 upper=0.78539816339744827899 effort=1000 velocity=1000.00 -> lower=-0.78539816339744827899 upper=0.78539816339744827899 effort=45 velocity=17.647
- joint rear_right_hip_y: limit lower=-0.89884456477707963539 upper=2.2951079663725435509 effort=1000 velocity=1000.00 -> lower=-0.89884456477707963539 upper=2.2951079663725435509 effort=45 velocity=17.647
- joint rear_right_knee: limit lower=-2.79253 upper=-0.261799 effort=1000 velocity=1000.00 -> lower=-2.7929 upper=-0.257725 effort=115 velocity=12.0

Commit message: Resolve config2 --> config typo

File: src/spot_skills/urdf/spot_with_arm.urdf (robot description, URDF)
Before this commit: robot spot, 24 links, 23 joints
Links:
- link arm_link_el0: geometry collision mesh filename=package://spot_description_noetic/meshes/arm/collision/arm_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; visual mesh filename=package://spot_description_noetic/meshes/arm/visual/arm_lin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
- link arm_link_el1: geometry collision mesh filename=package://spot_description_noetic/meshes/arm/collision/arm_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; collision mesh filename=package://spot_description_noetic/meshes/arm/collision/arm_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
- link arm_link_fngr: geometry collision mesh filename=package://spot_description_noetic/meshes/arm/collision/left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; collision mesh filename=package://spot_description_noetic/meshes/arm/collision/left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
- link arm_link_hr0: geometry collision mesh filename=package://spot_description_noetic/meshes/arm/collision/arm_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; visual mesh filename=package://spot_description_noetic/meshes/arm/visual/arm_lin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
- link arm_link_sh0: geometry collision mesh filename=package://spot_description_noetic/meshes/arm/collision/arm_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; collision mesh filename=package://spot_description_noetic/meshes/arm/collision/arm_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
- link arm_link_sh1: geometry visual mesh filename=package://spot_description_noetic/meshes/arm/visual/arm_lin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
- link arm_link_wr0: geometry collision mesh filename=package://spot_description_noetic/meshes/arm/collision/arm_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; visual mesh filename=package://spot_description_noetic/meshes/arm/visual/arm_lin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
- link arm_link_wr1: geometry collision mesh filename=package://spot_description_noetic/meshes/arm/collision/arm_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; collision mesh filename=package://spot_description_noetic/meshes/arm/collision/fron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
- link body: geometry collision mesh filename=package://spot_description_noetic/meshes/base/collision/bod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; visual mesh filename=package://spot_description_noetic/meshes/base/visual/body.o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
- link front_left_hip: geometry visual mesh filename=package://spot_description_noetic/meshes/base/visual/front_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
- link front_left_lower_leg: geometry collision mesh filename=package://spot_description_noetic/meshes/base/collision/lef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; collision sphere radius=0.036
- link front_left_upper_leg: geometry collision mesh filename=package://spot_description_noetic/meshes/base/collision/lef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; visual mesh filename=package://spot_description_noetic/meshes/base/visual/front_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
- link front_right_hip: geometry visual mesh filename=package://spot_description_noetic/meshes/base/visual/front_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
- link front_right_lower_leg: geometry collision mesh filename=package://spot_description_noetic/meshes/base/collision/rig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; collision sphere radius=0.036
- link front_right_upper_leg: geometry collision mesh filename=package://spot_description_noetic/meshes/base/collision/rig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; visual mesh filename=package://spot_description_noetic/meshes/base/visual/front_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
- link rear_left_hip: geometry visual mesh filename=package://spot_description_noetic/meshes/base/visual/rear_l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
- link rear_left_lower_leg: geometry collision mesh filename=package://spot_description_noetic/meshes/base/collision/lef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; collision sphere radius=0.036
- link rear_left_upper_leg: geometry collision mesh filename=package://spot_description_noetic/meshes/base/collision/lef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; visual mesh filename=package://spot_description_noetic/meshes/base/visual/rear_l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
- link rear_right_hip: geometry visual mesh filename=package://spot_description_noetic/meshes/base/visual/rear_r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
- link rear_right_lower_leg: geometry collision mesh filename=package://spot_description_noetic/meshes/base/collision/rig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; collision sphere radius=0.036
- link rear_right_upper_leg: geometry collision mesh filename=package://spot_description_noetic/meshes/base/collision/rig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; visual mesh filename=package://spot_description_noetic/meshes/base/visual/rear_r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
