Commit message: Apply MoveIt Setup Assistant to spot_moveit_config

File: src/spot_moveit_config/config/gazebo_spot.urdf (robot description, URDF)
Before this commit: robot spot, 24 links, 23 joints
Links:
- link arm_link_sh1: geometry collision mesh filename=package://spot_description/meshes/arm/visual/arm_link_sh1.o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; visual mesh filename=package://spot_description/meshes/arm/visual/arm_link_sh1.o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
- link front_left_hip: geometry collision mesh filename=package://spot_description/meshes/base/visual/front_left_hi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; visual mesh filename=package://spot_description/meshes/base/visual/front_left_hi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
- link front_right_hip: geometry collision mesh filename=package://spot_description/meshes/base/visual/front_right_h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; visual mesh filename=package://spot_description/meshes/base/visual/front_right_h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
- link rear_left_hip: geometry collision mesh filename=package://spot_description/meshes/base/visual/rear_left_hip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; visual mesh filename=package://spot_description/meshes/base/visual/rear_left_hip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
- link rear_right_hip: geometry collision mesh filename=package://spot_description/meshes/base/visual/rear_right_hi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; visual mesh filename=package://spot_description/meshes/base/visual/rear_right_hi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
